File: schematic/schematic.kicad_pcb (KiCad board)
At the start: 2 copper layers, 140 x 65 mm, 20 parts, among them J1 Conn_01x04_Pin, J2 Conn_01x08_Pin, SW1 SW_Push, SW2 SW_Push, U1 XIAO-ESP32-C3-SMD, U2 DHT11

Commit message: Finished customizing code and modified decorations of the PCB board.
Parts:
- removed the G*** at (127.5, 110.0)
- removed the G*** at (241.5, 110.5)
- added G***: LOGO, LOGO, F.Cu at (197.0, 112.0)
- added G***: LOGO, LOGO, F.Cu at (239.5, 118.0)
- added G***: LOGO, LOGO, F.Cu at (220.0, 103.0)
- added G***: LOGO, LOGO, F.Cu at (153.5, 96.0)
- added G***: LOGO, LOGO, F.Cu at (166.0, 116.5)
- added G***: LOGO, LOGO, F.Cu at (165.0, 108.0)
- added G***: LOGO, LOGO, F.Cu at (219.5, 117.0)
- added G***: LOGO, LOGO, F.Cu at (140.0, 110.5)
- added G***: LOGO, LOGO, F.Cu at (168.5, 68.0)
- added G***: LOGO, LOGO, F.Cu at (233.0, 106.0)
- added G***: LOGO, LOGO, F.Cu at (155.0, 80.5)
- added G***: LOGO, LOGO, F.Cu at (206.5, 72.5)
- added G***: LOGO, LOGO, F.Cu at (161.5, 99.0)
- added G***: LOGO, LOGO, F.Cu at (196.0, 127.5)
- added G***: LOGO, LOGO, F.Cu at (144.5, 120.0)
- added G***: LOGO, LOGO, F.Cu at (211.5, 75.5)
- added G***: LOGO, LOGO, F.Cu at (174.5, 119.0)
- added G***: LOGO, LOGO, F.Cu at (170.5, 100.5)
- added G***: LOGO, LOGO, F.Cu at (177.0, 65.0)
- added G***: LOGO, LOGO, F.Cu at (248.0, 116.0)
- added G***: LOGO, LOGO, F.Cu at (249.5, 109.0)
- added G***: LOGO, LOGO, F.Cu at (211.0, 128.0)
- added G***: LOGO, LOGO, F.Cu at (153.5, 121.5)
- added G***: LOGO, LOGO, F.Cu at (179.0, 103.0)
- added G***: LOGO, LOGO, F.Cu at (165.5, 131.5)
- added G***: LOGO, LOGO, F.Cu at (185.5, 62.5)
- added G***: LOGO, LOGO, F.Cu at (188.5, 129.5)
- added G***: LOGO, LOGO, F.Cu at (202.0, 100.5)
- added G***: LOGO, LOGO, F.Cu at (205.5, 115.5)
- added G***: LOGO, LOGO, F.Cu at (217.5, 86.5)
- added G***: LOGO, LOGO, F.Cu at (136.0, 117.0)
- added G***: LOGO, LOGO, F.Cu at (201.0, 66.5)
- added G***: LOGO, LOGO, F.Cu at (206.0, 107.0)
- added G***: LOGO, LOGO, F.Cu at (117.5, 109.5)
- added G***: LOGO, LOGO, F.Cu at (127.0, 115.5)
- added G***: LOGO, LOGO, F.Cu at (198.7, 86.7)
- added G***: LOGO, LOGO, F.Cu at (242.5, 101.5)
- added G***: LOGO, LOGO, F.Cu at (214.5, 111.0)
- added G***: LOGO, LOGO, F.Cu at (131.0, 100.0)
- added G***: LOGO, LOGO, F.Cu at (133.0, 108.0)
- added G***: LOGO, LOGO, F.Cu at (195.5, 104.0)
- added G***: LOGO, LOGO, F.Cu at (191.5, 110.0)
- added G***: LOGO, LOGO, F.Cu at (211.5, 99.0)
- added G***: LOGO, LOGO, F.Cu at (162.5, 73.0)
- added G***: LOGO, LOGO, F.Cu at (215.5, 80.5)
- added G***: LOGO, LOGO, F.Cu at (204.5, 129.0)
- added G***: LOGO, LOGO, F.Cu at (205.0, 122.5)
- added G***: LOGO, LOGO, F.Cu at (179.5, 128.0)
- added G***: LOGO, LOGO, F.Cu at (212.0, 121.0)
- added G***: LOGO, LOGO, F.Cu at (190.0, 117.0)
- added G***: LOGO, LOGO, F.Cu at (172.0, 94.5)
- added G***: LOGO, LOGO, F.Cu at (235.0, 97.5)
- added G***: LOGO, LOGO, F.Cu at (157.0, 128.0)
- added G***: LOGO, LOGO, F.Cu at (218.5, 125.0)
- added G***: LOGO, LOGO, F.Cu at (156.5, 105.5)
- added G***: LOGO, LOGO, F.Cu at (220.0, 93.5)
- added G***: LOGO, LOGO, F.Cu at (188.0, 104.5)
- added G***: LOGO, LOGO, F.Cu at (174.0, 109.5)
- added G***: LOGO, LOGO, F.Cu at (194.5, 65.0)
- added G***: LOGO, LOGO, F.Cu at (234.5, 120.5)
- added G***: LOGO, LOGO, F.Cu at (227.5, 101.0)
- added G***: LOGO, LOGO, F.Cu at (140.0, 101.5)
- added G***: LOGO, LOGO, F.Cu at (147.5, 104.0)
- added G***: LOGO, LOGO, F.Cu at (173.5, 86.5)
- added G***: LOGO, LOGO, F.Cu at (124.0, 106.5)
- added G***: LOGO, LOGO, F.Cu at (149.0, 112.0)
- added G***: LOGO, LOGO, F.Cu at (182.5, 111.5)
- added G***: LOGO, LOGO, F.Cu at (198.0, 119.5)
- added G***: LOGO, LOGO, F.Cu at (121.5, 113.0)
- added G***: LOGO, LOGO, F.Cu at (241.5, 110.0)
- added G***: LOGO, LOGO, F.Cu at (226.0, 120.5)
- added G***: LOGO, LOGO, F.Cu at (157.0, 115.0)
- added G***: LOGO, LOGO, F.Cu at (191.5, 97.9)
- added G***: LOGO, LOGO, F.Cu at (224.0, 110.0)
- added G***: LOGO, LOGO, F.Cu at (183.5, 120.5)
- added G***: LOGO, LOGO, F.Cu at (161.5, 124.0)
- added G***: LOGO, LOGO, F.Cu at (170.5, 125.5)
- added G***: LOGO, LOGO, F.Cu at (174.0, 130.5)
- added G***: LOGO, LOGO, F.Cu at (151.0, 87.5)
- added G***: LOGO, LOGO, F.Cu at (232.5, 114.0)
- added G***: LOGO, LOGO, B.Cu at (185.0, 86.7)
- moved J2 9.00 mm to (201.0, 105.8)
Routing:
- net /SDA: track 107.8 -> 60.1 mm
- net /SCL: track 82.3 -> 61.2 mm
- added copper zone on B.Cu, net GND
