File: schematic/schematic.kicad_pcb (KiCad board)
At the start: 2 copper layers, 140 x 65 mm, 99 parts, among them J1 Conn_01x04_Pin, J2 Conn_01x08_Pin, SW1 SW_Push, SW2 SW_Push, U1 XIAO-ESP32-C3-SMD, U2 DHT11

Commit message: Changed the orientation of the ESP32 to fit the UCB-C cable.
Parts:
- turned U1 to -90 degrees
Routing:
- net GND: track 203.7 -> 102.3 mm
- net /GPIO3: track 69.1 -> 44.0 mm
- net /GPIO2: track 89.0 -> 111.9 mm
- net +3.3V: track 98.0 -> 78.1 mm
- net /SCL: track 61.2 -> 52.7 mm
- net /DHT11 DATA: track 43.7 -> 45.9 mm
